Commit message: renamed vj

File: camera_tray/xacro/camera_tray.xacro (robot description, xacro)
@@ -9,5 +9,5 @@
         <!-- virtual joint -->
         <xacro:unless value="${not connected_to}">
-            <joint name="world" type="fixed">
+            <joint name="${prefix}_vj" type="fixed">
                 <parent link="${connected_to}" />
                 <child link="${prefix}_camera_fix" />

File: tray_gripper/xacro/tray_gripper.xacro (robot description, xacro)
@@ -9,5 +9,5 @@
         <!-- virtual joint -->
         <xacro:unless value="${not connected_to}">
-            <joint name="world" type="fixed">
+            <joint name="${prefix}_vj" type="fixed">
                 <parent link="${connected_to}" />
                 <child link="${prefix}_base_link" />
