Commit message: tcp added

File: tray_gripper/xacro/tray_gripper.xacro (robot description, xacro)
@@ -54,4 +54,21 @@
                 </geometry>
             </collision>
+        </link>
+        <joint
+            name="${prefix}_tcp_joint"
+            type="fixed">
+            <origin
+                xyz="0 -0.1345 0.225"
+                rpy="0 0 0" />
+            <parent
+                link="${prefix}_base_link" />
+            <child
+                link="${prefix}_tcp" />
+            <axis
+                xyz="0 0 0" />
+        </joint>
+        <link
+            name="${prefix}_tcp"
+        >
         </link>
         <link

Commit message: tray gripper updated

File: tray_gripper/xacro/tray_gripper.xacro (robot description, xacro)
@@ -1,181 +1,182 @@
 <?xml version="1.0"?>
 <robot xmlns:xacro="http://wiki.ros.org/xacro">
-    <xacro:macro name="tray_gripper"
-        params="
-        prefix:='tray_gripper'
-        connected_to:=''
-        *origin"
-    >
-        <!-- virtual joint -->
-        <xacro:unless value="${not connected_to}">
-            <joint name="${prefix}_vj" type="fixed">
-                <parent link="${connected_to}" />
-                <child link="${prefix}_base_link" />
-                <xacro:insert_block name="origin" />
-            </joint>
-        </xacro:unless>
-        <link
-            name="${prefix}_base_link">
-            <inertial>
-                <origin
-                    xyz="1.3918E-17 -0.0018924 0.010868"
-                    rpy="0 0 0" />
-                <mass
-                    value="1.6375" />
-                <inertia
-                    ixx="0.0013196"
-                    ixy="-3.504E-19"
-                    ixz="-1.2996E-18"
-                    iyy="0.0080644"
-                    iyz="-5.7578E-05"
-                    izz="0.009036" />
-            </inertial>
-            <visual>
-                <origin
-                    xyz="0 0 0"
-                    rpy="0 0 0" />
-                <geometry>
-                    <mesh
-                        filename="package://tray_gripper/meshes/gripper_base_link.STL" />
-                </geometry>
-                <material
-                    name="">
-                    <color
-                        rgba="0.64706 0.61961 0.58824 1" />
-                </material>
-            </visual>
-            <collision>
-                <origin
-                    xyz="0 0 0"
-                    rpy="0 0 0" />
-                <geometry>
-                    <mesh
-                        filename="package://tray_gripper/meshes/gripper_base_link.STL" />
-                </geometry>
-            </collision>
-        </link>
-        <joint
-            name="${prefix}_tcp_joint"
-            type="fixed">
-            <origin
-                xyz="0 -0.1345 0.225"
-                rpy="0 0 0" />
-            <parent
-                link="${prefix}_base_link" />
-            <child
-                link="${prefix}_tcp" />
-            <axis
-                xyz="0 0 0" />
-        </joint>
-        <link
-            name="${prefix}_tcp"
-        >
-        </link>
-        <link
-            name="${prefix}_rot">
-            <inertial>
-                <origin
-                    xyz="4.3535E-05 0.015829 0.063039"
-                    rpy="0 0 0" />
-                <mass
-                    value="3.8183" />
-                <inertia
-                    ixx="0.0020492"
-                    ixy="3.0924E-07"
-                    ixz="6.575E-06"
-                    iyy="0.019033"
-                    iyz="0.00014163"
-                    izz="0.019448" />
-            </inertial>
-            <visual>
-                <origin
-                    xyz="0 0 0"
-                    rpy="0 0 0" />
-                <geometry>
-                    <mesh
-                        filename="package://tray_gripper/meshes/gripper_rot.STL" />
-                </geometry>
-                <material
-                    name="">
-                    <color
-                        rgba="0.86667 0.86667 0.8902 1" />
-                </material>
-            </visual>
-            <collision>
-                <origin
-                    xyz="0 0 0"
-                    rpy="0 0 0" />
-                <geometry>
-                    <mesh
-                        filename="package://tray_gripper/meshes/gripper_rot.STL" />
-                </geometry>
-            </collision>
-        </link>
-        <joint
-            name="${prefix}_rot"
-            type="fixed">
-            <origin
-                xyz="0 -0.00036751 0.03766"
-                rpy="1.0472 0 0" />
-            <parent
-                link="${prefix}_base_link" />
-            <child
-                link="${prefix}_rot" />
-            <axis
-                xyz="0 0 0" />
-        </joint>
-        <link
-            name="${prefix}_camera">
-            <inertial>
-                <origin
-                    xyz="0 0 0"
-                    rpy="0 0 0" />
-                <mass
-                    value="0" />
-                <inertia
-                    ixx="0"
-                    ixy="0"
-                    ixz="0"
-                    iyy="0"
-                    iyz="0"
-                    izz="0" />
-            </inertial>
-            <visual>
-                <origin
-                    xyz="0 0 0"
-                    rpy="0 0 0" />
-                <geometry>
-                    <mesh
-                        filename="package://tray_gripper/meshes/gripper_camera.STL" />
-                </geometry>
-                <material
-                    name="">
-                    <color
-                        rgba="1 1 1 1" />
-                </material>
-            </visual>
-            <collision>
-                <origin
-                    xyz="0 0 0"
-                    rpy="0 0 0" />
-                <geometry>
-                    <mesh
-                        filename="package://tray_gripper/meshes/gripper_camera.STL" />
-                </geometry>
-            </collision>
-        </link>
-        <joint
-            name="${prefix}_camera"
-            type="fixed">
-            <origin
-                xyz="0 -0.0812 0.0263400000000001"
-                rpy="1.5707963267949 0 0" />
-            <parent
-                link="${prefix}_base_link" />
-            <child
-                link="${prefix}_camera" />
-            <axis
-                xyz="0 0 1" />
-        </joint>
-    </xacro:macro>
+  <xacro:macro name="tray_gripper"
+    params="
+      prefix:='tray_gripper'
+      connected_to:=''
+      *origin">
+    <!-- virtual joint -->
+    <xacro:unless value="${not connected_to}">
+      <joint name="${prefix}_vj" type="fixed">
+        <parent link="${connected_to}"/>
+        <child link="${prefix}_base_link"/>
+        <xacro:insert_block name="origin"/>
+      </joint>
+    </xacro:unless>
+    <!-- BASE -->
+    <link name="${prefix}_base_link">
+      <inertial>
+        <origin
+          xyz="1.54716176759448E-17 -0.00635902611918487 0.0126419354987282"
+          rpy="0 0 0"/>
+        <mass value="1.70056149639743"/>
+        <inertia
+          ixx="0.00148396285148825"
+          ixy="-3.79998537481848E-19"
+          ixz="-1.29772976157296E-18"
+          iyy="0.00807121460081302"
+          iyz="-3.97931642064587E-05"
+          izz="0.009194591178909"/>
+      </inertial>
+      <visual>
+        <origin xyz="0 0 0" rpy="0 0 0"/>
+        <geometry>
+          <mesh filename="package://tray_gripper/meshes/gripper_base_link.STL"/>
+        </geometry>
+        <material name="">
+          <color rgba="0.647058823529412 0.619607843137255 0.588235294117647 1"/>
+        </material>
+      </visual>
+      <collision>
+        <origin xyz="0 0 0" rpy="0 0 0"/>
+        <geometry>
+          <mesh filename="package://tray_gripper/meshes/gripper_base_link.STL"/>
+        </geometry>
+      </collision>
+    </link>
+    <!-- TCP -->
+    <joint name="${prefix}_tcp_joint" type="fixed">
+      <origin xyz="0 -0.1355 0.225" rpy="0 0 0"/>
+      <parent link="${prefix}_base_link"/>
+      <child link="${prefix}_tcp"/>
+    </joint>
+    <link name="${prefix}_tcp"/>
+    <!-- ROT -->
+    <link name="${prefix}_rot">
+      <inertial>
+        <origin
+          xyz="1.42155348395134E-16 0.0579058534888828 0.00661937034982867"
+          rpy="0 0 0"/>
+        <mass value="1.09080997852006"/>
+        <inertia
+          ixx="0.000647436272597154"
+          ixy="5.30862198661755E-18"
+          ixz="-6.26152856372176E-18"
+          iyy="0.0145519670294248"
+          iyz="-1.45418495884958E-06"
+          izz="0.0151280381685694"/>
+      </inertial>
+      <visual>
+        <origin xyz="0 0 0" rpy="0 0 0"/>
+        <geometry>
+          <mesh filename="package://tray_gripper/meshes/gripper_rot.STL"/>
+        </geometry>
+        <material name="">
+          <color rgba="0.866666666666667 0.866666666666667 0.890196078431372 1"/>
+        </material>
+      </visual>
+      <collision>
+        <origin xyz="0 0 0" rpy="0 0 0"/>
+        <geometry>
+          <mesh filename="package://tray_gripper/meshes/gripper_rot.STL"/>
+        </geometry>
+      </collision>
+    </link>
+    <joint name="${prefix}_rot" type="fixed">
+      <origin
+        xyz="0 -0.00036751 0.03766"
+        rpy="1.0472 0 0"/>
+      <parent link="${prefix}_base_link"/>
+      <child link="${prefix}_rot"/>
+    </joint>
+    <!-- CAMERA -->
+    <link name="${prefix}_camera">
+      <inertial>
+        <origin
+          xyz="0.00335751531690605 0.0146313170153883 -0.0879279715202068"
+          rpy="0 0 0"/>
+        <mass value="0.0270281785667234"/>
+        <inertia
+          ixx="4.82550992884901E-05"
+          ixy="-3.88228338689876E-06"
+          ixz="1.16964045190226E-05"
+          iyy="4.96884630389018E-05"
+          iyz="9.73483840232225E-06"
+          izz="8.82802544778306E-06"/>
+      </inertial>
+      <visual>
+        <origin xyz="0 0 0" rpy="0 0 0"/>
+        <geometry>
+          <mesh filename="package://tray_gripper/meshes/gripper_camera.STL"/>
+        </geometry>
+        <material name="">
+          <color rgba="1 1 1 1"/>
+        </material>
+      </visual>
+      <collision>
+        <origin xyz="0 0 0" rpy="0 0 0"/>
+        <geometry>
+          <mesh filename="package://tray_gripper/meshes/gripper_camera.STL"/>
+        </geometry>
+      </collision>
+    </link>
+    <joint name="${prefix}_camera" type="fixed">
+      <origin
+        xyz="0.003 -0.11282 0.017"
+        rpy="1.5708 0 0"/>
+      <parent link="${prefix}_base_link"/>
+      <child link="${prefix}_camera"/>
+    </joint>
+    <!-- <link
+        name="${prefix}_prod">
+        <inertial>
+        <origin
+            xyz="-0.078512151305398 -0.000462548063544956 0.00163585545247374"
+            rpy="0 0 0" />
+        <mass
+            value="0.143291460359673" />
+        <inertia
+            ixx="3.76239487433742E-05"
+            ixy="2.14711803634524E-07"
+            ixz="3.38112008987211E-06"
+            iyy="0.000133743724465417"
+            iyz="-8.4212870915275E-08"
+            izz="0.000165839633402877" />
+        </inertial>
+        <visual>
+        <origin
+            xyz="0 0 0"
+            rpy="0 0 0" />
+        <geometry>
+            <mesh
+            filename="package://tray_gripper/meshes/gripper_prod.STL" />
+        </geometry>
+        <material
+            name="">
+            <color
+            rgba="0.898039215686275 0.917647058823529 0.929411764705882 1" />
+        </material>
+        </visual>
+        <collision>
+        <origin
+            xyz="0 0 0"
+            rpy="0 0 0" />
+        <geometry>
+            <mesh
+            filename="package://tray_gripper/meshes/gripper_prod.STL" />
+        </geometry>
+        </collision>
+    </link>
+    <joint
+        name="${prefix}_prod"
+        type="fixed">
+        <origin
+            xyz="0 -0.1355 0.225"
+            rpy="-3.1416 -1.5361 1.5708" />
+        <parent
+            link="${prefix}_base_link" />
+        <child
+            link="${prefix}_prod" />
+    </joint> -->
+  </xacro:macro>
 </robot>
