Commit message: camera rotated

File: bucket_gripper/urdf/bucket_gripper.urdf (robot description, URDF)
Before this commit: robot bucket_gripper, 4 links, 3 joints
Joints:
- joint camera_joint: origin xyz=0.1845 0.0015 0.11707 rpy=0 0 0 -> xyz=0.1845 0.0015 0.11707 rpy=0 0 0.0

File: bucket_gripper/xacro/bucket_gripper.xacro (robot description, xacro)
@@ -134,5 +134,5 @@
     </joint>
     <joint name="${prefix}_camera_joint" type="fixed">
-      <origin xyz="0.1845 0.0015 0.11707" rpy="0 0 0" />
+      <origin xyz="0.1845 0.0015 0.11707" rpy="0 0 1.57" />
       <parent link="${prefix}_base_link" />
       <child  link="${prefix}_camera_link" />
