Commit message: update camera urdf

File: bucket_gripper/xacro/bucket_gripper.xacro (robot description, xacro)
@@ -22,5 +22,5 @@
     <link name="${prefix}_base_link">
       <inertial>
-        <origin xyz="-2.3651E-06 -4.3839E-06 0.063528" rpy="0 0 0" />
+        <origin xyz="5.6808E-06 -0.028248 0.061236" rpy="0 0 0" />
         <mass value="3.8087" />
         <inertia
@@ -47,5 +47,5 @@
     <link name="${prefix}_bucket_link">
       <inertial>
-        <origin xyz="8.4412E-15 2.092E-06 -0.05627" rpy="0 0 0" />
+        <origin xyz="9.1954E-15 3.7621E-06 -0.015079" rpy="0 0 0" />
         <mass value="1.124" />
         <inertia
@@ -72,5 +72,5 @@
     <link name="${prefix}_adapter_link">
       <inertial>
-        <origin xyz="-2.7992E-15 8.193E-16 -0.0044409" rpy="0 0 0" />
+        <origin xyz="-1.3884E-15 -6.3275E-15 0.0090197" rpy="0 0 0" />
         <mass value="0.40686" />
         <inertia
@@ -97,5 +97,5 @@
     <link name="${prefix}_camera_link">
       <inertial>
-        <origin xyz="0 0 0" rpy="0 0 0" />
+        <origin xyz="-0.0018857 0.006046 -0.019502" rpy="0 0 0" />
         <mass value="0" />
         <inertia
@@ -134,5 +134,5 @@
     </joint>
     <joint name="${prefix}_camera_joint" type="fixed">
-      <origin xyz="0.1845 0.0015 0.11707" rpy="0 0 1.57" />
+      <origin xyz="0.1215 0.0015 0.05332" rpy="0 0 1.5708" />
       <parent link="${prefix}_base_link" />
       <child  link="${prefix}_camera_link" />
